File: Cpu16_cad/Modulo_01_Reloj/Modulo_01_Reloj.kicad_sch (KiCad schematic)
At the start: 9 parts, among them SW1 SW_Rotary_1x3_MP, U1 TLC555xD

Commit message: mod reloj_cont
Parts:
- added C10, C11, C12, C13, C8, C9: 100nF, symbol Device:C
- added C2: 10nF, symbol Device:C
- added C3, C7: 1uF, symbol Device:C_Polarized
- added D1: 1N4148, Diode_THT:D_DO-35_SOD27_P7.62mm_Horizontal, symbol Diode:1N4148
- added D2: TL431LP, Package_TO_SOT_THT:TO-92_Inline, symbol Reference_Voltage:TL431LP
- added D3: LED, symbol Device:LED
- added R10, R12, R6, R9: 10k, symbol Device:R
- added R11: 1.5k, symbol Device:R
- added R13: 2.2k, symbol Device:R
- added R3, R8: 470k, symbol Device:R
- added R4: 4.7K, symbol Device:R
- added R5: 100k, symbol Device:R
- added R7: 12k, symbol Device:R
- added SW2, SW4: SW_Push, symbol Switch:SW_Push
- added SW3: SW_SPDT, symbol Switch:SW_SPDT
- added U2: TLC555xD, Package_SO:SOIC-8_3.9x4.9mm_P1.27mm, symbol Timer:TLC555xD
- added U3: 74HC00, symbol 74xx:74HC00
- added U4: 74HC04, symbol 74xx:74HC04
- added U5: 74HC74, symbol 74xx:74HC74
- added U6: 74HC14, symbol 74xx:74HC14
- added U8: LM393, symbol Comparator:LM393
Connections:
- net +5V: now also C10.1, C11.1, C12.1, C13.1, C9.1, D1.1 (K), R10.1, R11.1, R12.1, R3.2, R4.2, R5.1, R6.1, SW3.1 (A), U2.4 (~{RST}), U2.8 (VCC), U3.14 (VCC), U4.14 (VCC), U5.1 (~{R}), U5.10 (~{S}), U5.11 (C), U5.12 (D), U5.13 (~{R}), U5.14 (VCC), U5.4 (~{S}), U6.14 (VCC), U8.5 (+), U8.8 (V+)
- net ASTABLE: now also U3.1
- net GND: now also C10.2, C11.2, C12.2, C13.2, C2.1, C3.2, C7.2, C8.1, C9.2, D2.3 (K), D3.2 (A), R7.2, SW2.1, SW3.3 (C), SW4.2, U2.1 (GND), U3.7 (GND), U4.7 (GND), U5.7 (GND), U6.11, U6.13, U6.5, U6.7 (GND), U6.9, U8.4 (V-), U8.6 (-)
- new net: C8.2, R9.2, U2.2 (TRIG)
- new net: C2.2, U2.5 (CONT)
- new net: R10.2, R9.1, SW2.2
- new net: D3.1 (K), R13.2
- new net CLK_G: U3.11
- new net CLK_PRE: R13.1
- new net CLK_RAW: U3.12, U3.8, U4.9
- new net CLK_RAW_N: U4.8, U5.3 (C)
- new net HALT_N: R4.1, U5.2 (D)
- new net HALT_SYNC: U3.13, U5.5 (Q)
- new net MANUAL: U2.3 (OUT), U3.4
- new net MONO_C: C7.1, R3.1, U2.6 (THRES), U2.7 (DISCH)
- new net N1: U3.3, U3.9
- new net N2: U3.10, U3.6
- new net RESET_N: U6.4
- new net RST_A: U6.2, U6.3
- new net RST_RC: C3.1, D1.2 (A), R12.2, R5.2, R8.1, SW4.1, U6.1, U8.1
- new net SEL: SW3.2 (B), U3.5, U4.1
- new net SEL_N: U3.2, U4.2
- new net VREF: D2.1 (REF), D2.2 (A), R11.2, U8.2 (-)
- new net VSENSE: R6.2, R7.1, R8.2, U8.3 (+)
- no-connect marks 0 -> 8

Commit message: fix + revision
Parts:
- added C14, C15, C16: 100nF, symbol Device:C
- added C17: 47uF, symbol Device:C_Polarized
- added unit 5 of U4
- added unit 6 of U4
- added unit 2 of U4
- added unit 3 of U4
- added U7: 74HC244, symbol 74xx:74HC244
- C1, C5: value 10nf -> 10nF
- C4: value 1uf -> 1uF
- C6: value 1nf -> 1nF
- R11: value 1.5k -> 1k5
- R13: value 2.2k -> 2k2
- R4: value 4.7K -> 4k7
Connections:
- net +5V: now also C14.2, C15.1, C16.2, C17.1, U7.20 (VCC)
- net CLK: now also U7.12 (1Y3), U7.14 (1Y2), U7.16 (1Y1), U7.18 (1Y0)
- net CLK_N: now also U7.3 (2Y0), U7.5 (2Y1), U7.7 (2Y2), U7.9 (2Y3)
- net CLK_PRE: now also U4.5, U7.2 (1A0), U7.4 (1A1), U7.6 (1A2), U7.8 (1A3)
- net GND: now also C14.1, C15.2, C16.1, C17.2, U4.11, U4.13, U4.3, U7.1 (1OE), U7.10 (GND), U7.19 (2OE)
- new net CLK_N_PRE: U4.6, U7.11 (2A3), U7.13 (2A2), U7.15 (2A1), U7.17 (2A0)
- no-connect marks 8 -> 11
Other:
- sheet Coenctores renamed Conectores
- note added: "Modulo de Reloj para placa de 16 bits"
- note added: "Reloj V0.1a"
- moved on the sheet: U3D, U4D
